File: CN5501_LED_DRIVER.kicad_sch (KiCad schematic)
At the start: 5 parts

Commit message: finalised layout
Connections:
- net _INPUT_SUPPLY renamed _VIN
- net _VIN: no longer U?.2 (EN)
- new net _EN: U?.2 (EN)
Changed lines of the file:
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@@
 (kicad_sch (version 20230121) (generator eeschema)
   (paper "A4")
-  (junction (at 110.49 69.85) (diameter 0) (color 0 0 0 0)
-  )
   (junction (at 93.98 69.85) (diameter 0) (color 0 0 0 0)
-  )
-  (wire (pts (xy 110.49 82.55) (xy 110.49 69.85))
-    (stroke (width 0) (type default))
   )
   (wire (pts (xy 93.98 80.01) (xy 93.98 81.28))
@@
     (stroke (width 0) (type default))
   )
-  (wire (pts (xy 110.49 69.85) (xy 93.98 69.85))
-    (stroke (width 0) (type default))
-  )
-  (wire (pts (xy 121.92 69.85) (xy 110.49 69.85))
+  (wire (pts (xy 93.98 69.85) (xy 121.92 69.85))
     (stroke (width 0) (type default))
   )
@@
     (effects (font (size 1.27 1.27)) (justify right))
   )
-  (hierarchical_label "_INPUT_SUPPLY" (shape input) (at 88.9 69.85 180) (fields_autoplaced)
+  (hierarchical_label "_VIN" (shape input) (at 88.9 69.85 180) (fields_autoplaced)
     (effects (font (size 1.27 1.27)) (justify right))
   )
@@
     (effects (font (size 1.27 1.27)) (justify left))
   )
+  (hierarchical_label "_EN" (shape input) (at 110.49 82.55 180) (fields_autoplaced)
+    (effects (font (size 1.27 1.27)) (justify right))
+  )
   (hierarchical_label "_GND" (shape input) (at 121.92 105.41 270) (fields_autoplaced)
