File: UV_LED.kicad_pcb (KiCad board)
At the start: 2 copper layers, 369.6 x 24.1 mm, 33 parts, among them IC1 IS31LT3178-GRLS4-TR, J1 Conn_01x04, J2 Conn_01x04, Q1 Q_NMOS_GDS, Q2 Q_NMOS_GDS

Commit message: finalised layout
Parts:
- removed D12, D7: LED, LED_SMD:LED_1W_3W_R8
- removed D14, D15: 1N4001, Diode_SMD:D_SMA
- removed IC1: IS31LT3178-GRLS4-TR, Package_SO:HSOP-8-1EP_3.9x4.9mm_P1.27mm_EP2.41x3.1mm
- removed Q2: Q_NMOS_GDS, Package_TO_SOT_SMD:SOT-23
- added L1: 33 to 100 uH, Inductor_SMD:L_12x12mm_H4.5mm, F.Cu at (105.0, 117.5)
- added R4: R, Resistor_SMD:R_0603_1608Metric_Pad0.98x0.95mm_HandSolder, F.Cu at (100.0, 105.0)
- added TP1: TestPoint, TestPoint:TestPoint_THTPad_2.0x2.0mm_Drill1.0mm, F.Cu at (85.9, 29.4)
- added TP2: TestPoint, TestPoint:TestPoint_THTPad_2.0x2.0mm_Drill1.0mm, F.Cu at (85.9, 33.5)
- added TP3: TestPoint, TestPoint:TestPoint_THTPad_2.0x2.0mm_Drill1.0mm, F.Cu at (85.9, 37.5)
- added TP4: TestPoint, TestPoint:TestPoint_THTPad_2.0x2.0mm_Drill1.0mm, F.Cu at (85.9, 41.6)
- added TP5: TestPoint, TestPoint:TestPoint_THTPad_2.0x2.0mm_Drill1.0mm, F.Cu at (85.9, 45.6)
- added U1: ~, Package_TO_SOT_SMD:SOT-89-5_Handsoldering, F.Cu at (90.2, 113.0)
- C1: value 1n 50V -> 4,7 to 10 uF; footprint Capacitor_SMD:C_1206_3216Metric -> Capacitor_SMD:C_1210_3225Metric_Pad1.33x2.70mm_HandSolder
- C2: value 0,1 uF 50V -> 100nF; footprint Capacitor_SMD:C_1206_3216Metric -> Capacitor_SMD:C_0805_2012Metric_Pad1.18x1.45mm_HandSolder
- C3: value 0,1 uF 50V -> C; footprint Capacitor_SMD:C_1206_3216Metric -> Capacitor_SMD:C_1206_3216Metric_Pad1.33x1.80mm_HandSolder
- D1: value LED -> D_Schottky; footprint LED_SMD:LED_1W_3W_R8 -> Diode_SMD:D_SMA_Handsoldering
- D10, D11, D8, D9: value LED -> LED_Pad; footprint LED_SMD:LED_1W_3W_R8 -> meins:UV_3535
- D2, D3, D4, D5: footprint LED_SMD:LED_1W_3W_R8 -> LED_SMD:LED_1210_3225Metric_Pad1.42x2.65mm_HandSolder
- Q1: value Q_NMOS_GDS -> Q_NMOS_GSD
- R1, R2: value R -> Rs; footprint Resistor_SMD:R_1206_3216Metric -> Resistor_SMD:R_1206_3216Metric_Pad1.30x1.75mm_HandSolder
- R3: footprint Resistor_SMD:R_1206_3216Metric -> Resistor_SMD:R_2512_6332Metric_Pad1.40x3.35mm_HandSolder
- moved J2 323.2 mm to (80.3, 52.2), turned to 0 degrees
- moved R2 291.7 mm to (82.5, 113.0), turned to 90 degrees
- moved R1 291.6 mm to (77.5, 113.0), turned to 90 degrees
- moved H9 290.0 mm to (69.4, 47.3)
- moved C1 275.3 mm to (90.2, 121.9), turned to 0 degrees
- moved H4 270.1 mm to (61.5, 31.4), turned to 0 degrees
- moved Q1 264.3 mm to (105.0, 105.0), turned to 0 degrees
- moved D5 230.4 mm to (122.5, 107.5), turned to 0 degrees
- moved H8 224.1 mm to (69.4, 39.4)
- moved H3 206.3 mm to (53.5, 47.3), turned to 0 degrees
- moved D2 197.5 mm to (340.0, 107.5), turned to 0 degrees
- moved H7 162.2 mm to (69.4, 31.4)
- moved C3 158.2 mm to (229.9, 119.4), turned to 0 degrees
- moved H2 146.8 mm to (53.5, 39.4), turned to 0 degrees
- moved H1 102.4 mm to (53.5, 31.4), turned to 0 degrees
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Connections:
- C1 pad 1: Net-(IC1-Pad1) -> +36V
- C3 pad 1: +36V -> UV_LED+
- C3 pad 2: GND -> UV_LED-
- D1 pad 1: Net-(D1-Pad1) -> +36V
- D10 pad 1: Net-(D11-Pad2) -> Net-(D10-K)
- D10 pad 2: Net-(D9-Pad1) -> Net-(D10-A)
- D10 pad 3: (no net) -> unconnected-(D10-PAD-Pad3)
- D11 pad 1: Net-(D11-Pad1) -> Net-(D10-A)
- D11 pad 2: Net-(D11-Pad2) -> UV_LED+
- D11 pad 3: (no net) -> unconnected-(D11-PAD-Pad3)
- D2 pad 2: Net-(D1-Pad1) -> Net-(D2-A)
- D5 pad 1: Net-(Q1-Pad2) -> Net-(D5-K)
- D8 pad 1: Net-(D9-Pad2) -> UV_LED-
- D8 pad 2: Net-(D7-Pad1) -> Net-(D8-A)
- D8 pad 3: (no net) -> unconnected-(D8-PAD-Pad3)
- D9 pad 1: Net-(D9-Pad1) -> Net-(D8-A)
- D9 pad 2: Net-(D9-Pad2) -> Net-(D10-K)
- D9 pad 3: (no net) -> unconnected-(D9-PAD-Pad3)
- Q1 pad 1: Net-(Q1-Pad1) -> Net-(Q1-G)
- Q1 pad 2: Net-(Q1-Pad2) -> GND
- Q1 pad 3: Net-(IC1-Pad1) -> Net-(D5-K)
- R1 pad 1: /TOGGLE -> +36V
- R1 pad 2: Net-(Q1-Pad1) -> UV_LED+
- R2 pad 1: Net-(Q1-Pad2) -> +36V
- R2 pad 2: Net-(Q2-Pad1) -> UV_LED+
- R3 pad 1: Net-(IC1-Pad4) -> Net-(D2-A)
- R3 pad 2: GND -> +36V
Routing:
- net /PWM: track 409.8 -> 0.00 mm, vias 1 -> 0
- net /TOGGLE: track 378.8 -> 0.00 mm, vias 1 -> 0
- net GND: track 129.5 -> 0.00 mm, vias 59 -> 0
- net Net-(D11-Pad1): track 62.2 -> 0.00 mm
- net Net-(D4-K): track 58.4 -> 0.00 mm
- net Net-(D3-K): track 58.4 -> 0.00 mm
- net Net-(D2-K): track 58.4 -> 0.00 mm
- net Net-(D9-Pad1): track 58.4 -> 0.00 mm
- net Net-(D1-Pad1): track 58.4 -> 0.00 mm
- net Net-(D7-Pad1): track 58.4 -> 0.00 mm
- net Net-(D9-Pad2): track 58.4 -> 0.00 mm
- net Net-(D11-Pad2): track 58.4 -> 0.00 mm
- net +36V: track 33.2 -> 0.00 mm
- net Net-(D12-Pad1): track 25.9 -> 0.00 mm
- net Net-(IC1-Pad1): track 19.9 -> 0.00 mm
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- removed copper zone on B.Cu, net +36V
- removed copper zone on F.Cu, net GND
Other:
- board size 369.6 x 24.1 mm -> 333.1 x 26.4 mm
